Commit message: rework (same)

File: urdf/franka_robot.xacro (robot description, xacro)
@@ -1,5 +1,5 @@
 <?xml version='1.0' encoding='utf-8'?>
 <robot xmlns:xacro="http://www.ros.org/wiki/xacro">
-  <xacro:macro name="franka_robot" params="arm_id qbhand joint_limits">
+  <xacro:macro name="franka_robot" params="arm_id joint_limits">
     <!-- Name of this panda -->
     <!-- Should a franka_gripper be mounted at the flange?" -->
@@ -9,10 +9,10 @@
     <!-- Rotational offset between $(arm_id)_hand -> $(arm_id)_hand_tcp [rad]. Only used when hand:=true -->
     <xacro:arg name="tcp_rpy" default="0 0 0" />
-    <!-- Is the robot being simulated in gazebo? -->
+    <!-- Is the robot being simulated in gazebo?" -->
     <xacro:arg name="gazebo" default="false" />
     <!-- Qb hand parameters -->
-    <!-- Transform frame -->
-    <xacro:arg name="tcp_xyz_qb" default="0.1 -0.1 0.05" />
-    <xacro:arg name="tcp_rpy_qb" default="3.1416 -1.5708 -0.7854" />
+    <!-- Transform frame panda_link8 -> base_link_qbhand  first rotation then translation -->
+    <xacro:arg name="tcp_xyz_qb" default="0.1 0.0 0.0" />
+    <xacro:arg name="tcp_rpy_qb" default="0.0 0.0 -0.7854" />
     <xacro:include filename="$(find franka_description)/robots/common/utils.xacro" />
     <xacro:include filename="$(find franka_description)/robots/common/franka_arm.xacro" />
@@ -27,9 +27,11 @@
           connected_to="$(arg arm_id)_link8"
           safety_distance="0.03"
-          gazebo="$(arg gazebo)"/>
+          gazebo="$(arg gazebo)"
+       />
     </xacro:if>
     <xacro:if value="$(arg qbhand)">
       <xacro:include filename="$(find franka_qbhand)/urdf/softhands.xacro"/>
-      <xacro:softhands type="right"
+      <xacro:softhands
+        type="right"
         version="v2.0_simple"
         parent="$(arg arm_id)_link8"
@@ -37,5 +39,7 @@
         orientation="$(arg tcp_rpy_qb)"
         operation_mode="0"
-        translation="0.0036"/>
+        translation="0.0036"
+        gazebo="$(arg gazebo)"
+        />
     </xacro:if>
     <!-- Define additional Gazebo tags -->

File: urdf/panda.urdf.xacro (robot description, xacro)
@@ -3,7 +3,5 @@
   <xacro:include filename="$(find franka_qbhand)/urdf/franka_robot.xacro"/>
   <xacro:arg name="arm_id" default="panda" />
-  <xacro:arg name="qbhand" default="true" />
   <xacro:franka_robot arm_id="$(arg arm_id)"
-                      qbhand="$(arg qbhand)"
                       joint_limits="${xacro.load_yaml('$(find franka_description)/robots/panda/joint_limits.yaml')}">
   </xacro:franka_robot>

File: urdf/softhands.xacro (robot description, xacro)
@@ -42,5 +42,5 @@
   <xacro:include filename="$(find softhands_description)/urdf/v2.0/sh_v2.xacro"/>
   <xacro:include filename="$(find softhands_description)/urdf/v2.0_simple/sh_v2_simple.xacro"/>
-  <xacro:macro name="softhands" params="type version parent position orientation operation_mode translation">
+  <xacro:macro name="softhands" params="type version parent position orientation operation_mode translation gazebo:=true safety_distance:=0 description_pkg:=franka_description">
     # Softhand VERSION 1.0
     <xacro:if value="${version == 'v1.0'}">
@@ -72,8 +72,46 @@
     # Softhand VERSION 2.0 SIMPLIFIED (less joints)
     <xacro:if value="${version == 'v2.0_simple'}">
+      <link name="qbhand_flange0">
+        <visual>
+          <geometry>
+            <box size="30e-3 30e-3 30e-3" />
+          </geometry>
+        </visual>
+        <collision>
+          <origin xyz="30e-3 30e-3 30e-3" rpy="0 0 0" />
+          <geometry>
+            <box size="17.5e-3 15.2e-3 18.5e-3" />
+          </geometry>
+        </collision>
+      </link>
+      <link name="qbhand_flange1">
+        <visual>
+          <geometry>
+            <box size="30e-3 30e-3 30e-3" />
+          </geometry>
+        </visual>
+        <collision>
+          <origin xyz="30e-3 30e-3 30e-3" rpy="0 0 0" />
+          <geometry>
+            <box size="17.5e-3 15.2e-3 18.5e-3" />
+          </geometry>
+        </collision>
+      </link>
+      <!-- Create flange link -->
+      <joint name="qbhand_flange_joint0" type="fixed">
+        <parent link="${parent}" />
+        <child link="qbhand_flange0" />
+        <origin xyz="0 0 0" rpy="${orientation}" />
+      </joint>
+      <!-- Create end flange link -->
+      <joint name="qbhand_flange_joint1" type="fixed">
+        <parent link="qbhand_flange0" />
+        <child link="qbhand_flange1" />
+        <origin xyz="${position}" rpy="0 0 0" />
+      </joint>
       <xacro:sh_v2_simple type="${type}"
-	      parent = "${parent}"
-	      position ="${position}"
-	      orientation ="${orientation}"
+	      parent = "qbhand_flange1"
+	      position ="0 0 0"
+	      orientation ="3.14158 -1.5708 0"
         operation_mode = "${operation_mode}"
         translation="${translation}">
