Commit message: formatting

File: urdf/sh_v2_simple.xacro (robot description, xacro)
@@ -38,7 +38,7 @@
 -->
 <robot name="softhand_v2.0" xmlns:xacro="http://www.ros.org/wiki/xacro">
-  <xacro:include filename="$(find softhands_description)/urdf/v2.0_simple/finger.xacro"/>
-  <xacro:include filename="$(find softhands_description)/urdf/v2.0_simple/thumb.xacro"/>
-  <xacro:macro name="sh_v2_simple" params="type parent position orientation operation_mode translation">
+	<xacro:include filename="$(find softhands_description)/urdf/v2.0_simple/finger.xacro"/>
+	<xacro:include filename="$(find softhands_description)/urdf/v2.0_simple/thumb.xacro"/>
+	<xacro:macro name="sh_v2_simple" params="type parent position orientation operation_mode translation">
 	<material name="gray">
 		<color rgba="0.75 0.75 0.75 1"/>
@@ -54,42 +54,42 @@
     # RIGHT HAND
     <xacro:if value="${type == 'right'}">
-      # Palm
-      <joint name="${type}_hand_v2s_palm_joint" type="fixed">
-	      <origin xyz="0 0 0.00" rpy="0 -1.57 3.14159"/>
-	      <parent link="${type}_hand_v2s_palm_base" />
-	      <child link="${type}_hand_v2s_palm_link" />
-      </joint>
-      <link name="${type}_hand_v2s_palm_link">
-	<inertial>
-	  <origin xyz="-0.004568758 -0.006808116 0.027653328"/>
-	  <mass value="0.266"/>
-	  <inertia ixx="0.001" ixy="0" ixz="0" iyy="0.001" iyz="0" izz="0.001"/>
-	</inertial>
-	<visual>
-	  <geometry>
-	    <mesh filename="package://softhands_description/meshes/softhands/v2.0/right/qbh_palm_ng.stl" scale="0.001 0.001 0.001"/>
-	  </geometry>
-	  <material name="gray">
-+	  </material>
-	  </visual>
-	<collision>
-	  <geometry>
-	    <mesh filename="package://softhands_description/meshes/softhands/v2.0/right/qbh_palm_ng.stl" scale="0.001 0.001 0.001"/>
-	  </geometry>
-	</collision>
-      </link>
-      <gazebo reference="${type}_hand_v2s_palm_link">
-      <material>Gazebo/Grey</material>
-      <selfCollide>true</selfCollide>
+		# Palm
+		<joint name="${type}_hand_v2s_palm_joint" type="fixed">
+			<origin xyz="0 0 0.00" rpy="0 -1.57 3.14159"/>
+			<parent link="${type}_hand_v2s_palm_base" />
+			<child link="${type}_hand_v2s_palm_link" />
+     	</joint>
+	<link name="${type}_hand_v2s_palm_link">
+		<inertial>
+			<origin xyz="-0.004568758 -0.006808116 0.027653328"/>
+			<mass value="0.266"/>
+			<inertia ixx="0.001" ixy="0" ixz="0" iyy="0.001" iyz="0" izz="0.001"/>
+		</inertial>
+		<visual>
+			<geometry>
+				<mesh filename="package://softhands_description/meshes/softhands/v2.0/right/qbh_palm_ng.stl" scale="0.001 0.001 0.001"/>
+			</geometry>
+			<material name="gray">
+			</material>
+		</visual>
+		<collision>
+			<geometry>
+				<mesh filename="package://softhands_description/meshes/softhands/v2.0/right/qbh_palm_ng.stl" scale="0.001 0.001 0.001"/>
+			</geometry>
+		</collision>
+	</link>
+	<gazebo reference="${type}_hand_v2s_palm_link">
+		<material>Gazebo/Grey</material>
+		<selfCollide>true</selfCollide>
     </gazebo>
-      # Thumb finger
-      <xacro:thumb_v2_simple type="thumb"
-	      ns = "${type}_hand_v2s"
-	      sign = "-1"
-	      position="0.06643 -0.0437097 0.0210"
-	      orientation="-1.5707963 -0.7 -1.0471972"
-	      damping="0.05"
-	      translation="${translation}"> <!-- added offset on orientation -->
-      </xacro:thumb_v2_simple>
+	# Thumb finger
+	<xacro:thumb_v2_simple type="thumb"
+		ns = "${type}_hand_v2s"
+		sign = "-1"
+		position="0.06643 -0.0437097 0.0210"
+		orientation="-1.5707963 -0.7 -1.0471972"
+		damping="0.05"
+		translation="${translation}"> <!-- added offset on orientation -->
+	</xacro:thumb_v2_simple>
       # Index finger
       <xacro:finger_v2_simple type="index"
@@ -208,62 +208,62 @@
 	  # Gazebo NEW custom synergy-plugin
 	  <gazebo>
-	          <plugin name="synergy_plugin" filename="libsofthand_plugin.so">
-	                      <namespace>${type}_hand_v2s</namespace>
-	                      <operation_mode>${operation_mode}</operation_mode>
-	                      <!-- Optional parameter to fit with the real EGO's arm -->
-	                      <r_finger>0.0033</r_finger>
-	                      <R_pulley>0.0053</R_pulley>
-	                      <n_param>0.058</n_param> <!-- The formula is (4*r_finger)/(2*R_pulley) -->
-	                      <spring_k>0.5</spring_k>
-	                      <!-- Parameters for synergy matrix (S) -->
-	                      <synS_thumb_j1>1.2</synS_thumb_j1>
-	                      <synS_thumb_j2>1.2</synS_thumb_j2>
-	                      <synS_thumb_j3>1.2</synS_thumb_j3>
-	                      <k_thumb_j1>0.8</k_thumb_j1>
-	                      <k_thumb_j2>0.8</k_thumb_j2>
-	                      <k_thumb_j3>0.8</k_thumb_j3>
-	                      <synS_index_j2>1.57</synS_index_j2>
-	                      <synS_index_j3>1.25</synS_index_j3>
-	                      <synS_index_j4>0.8</synS_index_j4>
-	                      <k_index_j1>0.25</k_index_j1>
-	                      <k_index_j2>0.5</k_index_j2>
-	                      <k_index_j3>0.5</k_index_j3>
-	                      <k_index_j4>0.5</k_index_j4>
-	                      <synS_middle_j2>1.57</synS_middle_j2>
-	                      <synS_middle_j3>1.25</synS_middle_j3>
-	                      <synS_middle_j4>1.25</synS_middle_j4>
-	                      <k_middle_j1>0.25</k_middle_j1>
-	                      <k_middle_j2>0.5</k_middle_j2>
-	                      <k_middle_j3>0.5</k_middle_j3>
-	                      <k_middle_j4>0.5</k_middle_j4>
-	                      <synS_ring_j2>1.57</synS_ring_j2>
-	                      <synS_ring_j3>1.0</synS_ring_j3>
-	                      <synS_ring_j4>1.0</synS_ring_j4>
-	                      <k_ring_j1>0.25</k_ring_j1>
-	                      <k_ring_j2>0.5</k_ring_j2>
-	                      <k_ring_j3>0.5</k_ring_j3>
-	                      <k_ring_j4>0.5</k_ring_j4>
-	                      <synS_little_j2>1.57</synS_little_j2>
-	                      <synS_little_j3>1.25</synS_little_j3>
-	                      <synS_little_j4>1.0</synS_little_j4>
-	                      <k_little_j1>0.25</k_little_j1>
-	                      <k_little_j2>0.5</k_little_j2>
-	                      <k_little_j3>0.5</k_little_j3>
-	                      <k_little_j4>0.5</k_little_j4>
-	                     	# Change tags sign according to the hand type
-												<xacro:if value="${type == 'right'}">
-														<synS_index_j1>0.3</synS_index_j1>
-														<synS_middle_j1>0</synS_middle_j1>
-														<synS_ring_j1>0</synS_ring_j1>
-														<synS_little_j1>-0.2</synS_little_j1>
-                      	</xacro:if>
-												<xacro:if value="${type == 'left'}">
-														<synS_index_j1>-0.3</synS_index_j1>
-														<synS_middle_j1>0</synS_middle_j1>
-														<synS_ring_j1>0</synS_ring_j1>
-														<synS_little_j1>0.1</synS_little_j1>
-                      	</xacro:if>
-	          </plugin>
-	  </gazebo>
-  </xacro:macro>
+			<plugin name="synergy_plugin" filename="libsofthand_plugin.so">
+				<namespace>${type}_hand_v2s</namespace>
+				<operation_mode>${operation_mode}</operation_mode>
+				<!-- Optional parameter to fit with the real EGO's arm -->
+				<r_finger>0.0033</r_finger>
+				<R_pulley>0.0053</R_pulley>
+				<n_param>0.058</n_param> <!-- The formula is (4*r_finger)/(2*R_pulley) -->
+				<spring_k>0.5</spring_k>
+				<!-- Parameters for synergy matrix (S) -->
+				<synS_thumb_j1>1.2</synS_thumb_j1>
+				<synS_thumb_j2>1.2</synS_thumb_j2>
+				<synS_thumb_j3>1.2</synS_thumb_j3>
+				<k_thumb_j1>0.8</k_thumb_j1>
+				<k_thumb_j2>0.8</k_thumb_j2>
+				<k_thumb_j3>0.8</k_thumb_j3>
+				<synS_index_j2>1.57</synS_index_j2>
+				<synS_index_j3>1.25</synS_index_j3>
+				<synS_index_j4>0.8</synS_index_j4>
+				<k_index_j1>0.25</k_index_j1>
+				<k_index_j2>0.5</k_index_j2>
+				<k_index_j3>0.5</k_index_j3>
+				<k_index_j4>0.5</k_index_j4>
+				<synS_middle_j2>1.57</synS_middle_j2>
+				<synS_middle_j3>1.25</synS_middle_j3>
+				<synS_middle_j4>1.25</synS_middle_j4>
+				<k_middle_j1>0.25</k_middle_j1>
+				<k_middle_j2>0.5</k_middle_j2>
+				<k_middle_j3>0.5</k_middle_j3>
+				<k_middle_j4>0.5</k_middle_j4>
+				<synS_ring_j2>1.57</synS_ring_j2>
+				<synS_ring_j3>1.0</synS_ring_j3>
+				<synS_ring_j4>1.0</synS_ring_j4>
+				<k_ring_j1>0.25</k_ring_j1>
+				<k_ring_j2>0.5</k_ring_j2>
+				<k_ring_j3>0.5</k_ring_j3>
+				<k_ring_j4>0.5</k_ring_j4>
+				<synS_little_j2>1.57</synS_little_j2>
+				<synS_little_j3>1.25</synS_little_j3>
+				<synS_little_j4>1.0</synS_little_j4>
+				<k_little_j1>0.25</k_little_j1>
+				<k_little_j2>0.5</k_little_j2>
+				<k_little_j3>0.5</k_little_j3>
+				<k_little_j4>0.5</k_little_j4>
+				# Change tags sign according to the hand type
+				<xacro:if value="${type == 'right'}">
+					<synS_index_j1>0.3</synS_index_j1>
+					<synS_middle_j1>0</synS_middle_j1>
+					<synS_ring_j1>0</synS_ring_j1>
+					<synS_little_j1>-0.2</synS_little_j1>
+				</xacro:if>
+				<xacro:if value="${type == 'left'}">
+					<synS_index_j1>-0.3</synS_index_j1>
+					<synS_middle_j1>0</synS_middle_j1>
+					<synS_ring_j1>0</synS_ring_j1>
+					<synS_little_j1>0.1</synS_little_j1>
+				</xacro:if>
+			</plugin>
+		</gazebo>
+	</xacro:macro>
 </robot>
