Commit message: restarted ros files

File: urdf/franka_robot_qb.xacro (robot description, xacro)
@@ -11,8 +11,4 @@
     <!-- Is the robot being simulated in gazebo?" -->
     <xacro:arg name="gazebo" default="false" />
-    <!-- Qb hand parameters -->
-    <!-- Transform frame panda_link8 -> base_link_qbhand  first rotation then translation -->
-    <xacro:arg name="tcp_xyz_qb" default="0.1 0.0 0.0" />
-    <xacro:arg name="tcp_rpy_qb" default="0.0 0.0 -0.7854" />
     <xacro:include filename="$(find franka_description)/robots/common/utils.xacro" />
     <xacro:include filename="$(find franka_description)/robots/common/franka_arm.xacro" />
@@ -30,16 +26,15 @@
        />
     </xacro:if>
-    <xacro:if value="$(arg qbhand)">
+    <xacro:if value="$(arg use_qbhand)">
       <xacro:include filename="$(find franka_qbhand)/urdf/softhands.xacro"/>
       <xacro:softhands
-        type="right"
-        version="v2.0_simple"
-        parent="$(arg arm_id)_link8"
-        position="$(arg tcp_xyz_qb)"
-        orientation="$(arg tcp_rpy_qb)"
-        operation_mode="0"
+        type = "right"
+        version = "v2.0_simple"
+        parent = "panda_link8"
+        position ="0 0 0"
+        orientation ="0 0 0"
+        operation_mode = "0"
         translation="0.0036"
-        gazebo="$(arg gazebo)"
-        />
+      />
     </xacro:if>
     <!-- Define additional Gazebo tags -->

File: urdf/panda_qb.urdf.xacro (robot description, xacro)
@@ -1,5 +1,5 @@
 <?xml version='1.0' encoding='utf-8'?>
 <robot xmlns:xacro="http://www.ros.org/wiki/xacro" name="panda">
-  <xacro:include filename="$(find franka_qbhand)/urdf/franka_robot.xacro"/>
+  <xacro:include filename="$(find franka_qbhand)/urdf/franka_robot_qb.xacro"/>
   <xacro:arg name="arm_id" default="panda" />
   <xacro:franka_robot arm_id="$(arg arm_id)"

File: urdf/softhands.xacro (robot description, xacro)
@@ -38,85 +38,14 @@
 -->
 <robot name="softhands" xmlns:xacro="http://www.ros.org/wiki/xacro">
-  <xacro:include filename="$(find softhands_description)/urdf/v1.0/sh_v1.xacro"/>
-  <xacro:include filename="$(find softhands_description)/urdf/v1.0_simple/sh_v1_simple.xacro"/>
-  <xacro:include filename="$(find softhands_description)/urdf/v2.0/sh_v2.xacro"/>
-  <xacro:include filename="$(find softhands_description)/urdf/v2.0_simple/sh_v2_simple.xacro"/>
-  <xacro:macro name="softhands" params="type version parent position orientation operation_mode translation gazebo:=true safety_distance:=0 description_pkg:=franka_description">
-    # Softhand VERSION 1.0
-    <xacro:if value="${version == 'v1.0'}">
-    	<xacro:sh_v1 type="${type}"
-    	    parent = "${parent}"
-    	    position ="${position}"
-    	    orientation ="${orientation}"
-          operation_mode = "${operation_mode}">
-    	</xacro:sh_v1>
-    </xacro:if>
-    # Softhand VERSION 1.0 SIMPLIFIED (less joints)
-    <xacro:if value="${version == 'v1.0_simple'}">
-      <xacro:sh_v1_simple type="${type}"
-        parent = "${parent}"
-        position ="${position}"
-        orientation ="${orientation}"
-        operation_mode = "${operation_mode}">
-      </xacro:sh_v1_simple>
-    </xacro:if>
-    # Softhand VERSION 2.0
-    <xacro:if value="${version == 'v2.0'}">
-      <xacro:sh_v2 type="${type}"
-	      parent = "${parent}"
-	      position ="${position}"
-	      orientation ="${orientation}"
-        operation_mode = "${operation_mode}">
-      </xacro:sh_v2>
-    </xacro:if>
+  <xacro:include filename="$(find franka_qbhand)/urdf/sh_v2_simple.xacro"/>
+  <xacro:macro name="softhands" params="type version parent position orientation operation_mode translation">
     # Softhand VERSION 2.0 SIMPLIFIED (less joints)
-    <xacro:if value="${version == 'v2.0_simple'}">
-      <link name="qbhand_flange0">
-        <visual>
-          <geometry>
-            <box size="30e-3 30e-3 30e-3" />
-          </geometry>
-        </visual>
-        <collision>
-          <origin xyz="30e-3 30e-3 30e-3" rpy="0 0 0" />
-          <geometry>
-            <box size="17.5e-3 15.2e-3 18.5e-3" />
-          </geometry>
-        </collision>
-      </link>
-      <link name="qbhand_flange1">
-        <visual>
-          <geometry>
-            <box size="30e-3 30e-3 30e-3" />
-          </geometry>
-        </visual>
-        <collision>
-          <origin xyz="30e-3 30e-3 30e-3" rpy="0 0 0" />
-          <geometry>
-            <box size="17.5e-3 15.2e-3 18.5e-3" />
-          </geometry>
-        </collision>
-      </link>
-      <!-- Create flange link -->
-      <joint name="qbhand_flange_joint0" type="fixed">
-        <parent link="${parent}" />
-        <child link="qbhand_flange0" />
-        <origin xyz="0 0 0" rpy="${orientation}" />
-      </joint>
-      <!-- Create end flange link -->
-      <joint name="qbhand_flange_joint1" type="fixed">
-        <parent link="qbhand_flange0" />
-        <child link="qbhand_flange1" />
-        <origin xyz="${position}" rpy="0 0 0" />
-      </joint>
-      <xacro:sh_v2_simple type="${type}"
-	      parent = "qbhand_flange1"
-	      position ="0 0 0"
-	      orientation ="3.14158 -1.5708 0"
-        operation_mode = "${operation_mode}"
-        translation="${translation}">
-      </xacro:sh_v2_simple>
-    </xacro:if>
-    # TODO: OTHER VERSIONs
+    <xacro:sh_v2_simple type="${type}"
+      parent = "${parent}"
+      position ="${position}"
+      orientation ="${orientation}"
+      operation_mode = "${operation_mode}"
+      translation="${translation}">
+    </xacro:sh_v2_simple>
     <gazebo>
       <self_collide>1</self_collide>

Commit message: mass compensation

File: urdf/franka_robot_qb.xacro (robot description, xacro)
@@ -11,4 +11,8 @@
     <!-- Is the robot being simulated in gazebo?" -->
     <xacro:arg name="gazebo" default="false" />
+    <!-- Positional offset between $(arm_id)_hand -> $(arm_id)_hand_tcp [m]. Only used when hand:=true -->
+    <xacro:arg name="qb_tcp_xyz" default="0.12 0 0.05" />
+    <!-- Rotational offset between $(arm_id)_hand -> $(arm_id)_hand_tcp [rad]. Only used when hand:=true -->
+    <xacro:arg name="qb_tcp_rpy" default="0 -1.5707963 2.3561944" />
     <xacro:include filename="$(find franka_description)/robots/common/utils.xacro" />
     <xacro:include filename="$(find franka_description)/robots/common/franka_arm.xacro" />
@@ -27,4 +31,28 @@
     </xacro:if>
     <xacro:if value="$(arg use_qbhand)">
+      <joint name="mass_compensation_joint" type="fixed">
+	      <origin xyz="-0.12 0 0.05" rpy="0 0 0"/>
+	      <parent link="panda_link8" />
+	      <child link="mass_compensation_link" />
+      </joint>
+      <link name="mass_compensation_link">
+        <inertial>
+          <origin xyz="0 0 0"/>
+          <mass value="0.76"/>
+          <inertia ixx="0.01" ixy="0" ixz="0" iyy="0.01" iyz="0" izz="0.01"/>
+        </inertial>
+        <visual>
+          <geometry>
+            <box size="0.1 0.1 0.1"/>
+          </geometry>
+          <material name="gray">
+    +	  </material>
+        </visual>
+        <collision>
+          <geometry>
+            <box size="0.1 0.1 0.1"/>
+          </geometry>
+        </collision>
+      </link>
       <xacro:include filename="$(find franka_qbhand)/urdf/softhands.xacro"/>
       <xacro:softhands
@@ -32,6 +60,6 @@
         version = "v2.0_simple"
         parent = "panda_link8"
-        position ="0.12 0 0.05"
-        orientation ="0 -1.5707963 2.3561944"
+        position ="$(arg qb_tcp_xyz)"
+        orientation ="$(arg qb_tcp_xyz)"
         operation_mode = "0"
         translation="0.0036"

Commit message: fixed rotation and compensation

File: urdf/franka_robot_qb.xacro (robot description, xacro)
@@ -14,5 +14,5 @@
     <xacro:arg name="qb_tcp_xyz" default="0.12 0 0.05" />
     <!-- Rotational offset between $(arm_id)_hand -> $(arm_id)_hand_tcp [rad]. Only used when hand:=true -->
-    <xacro:arg name="qb_tcp_rpy" default="0 -1.5707963 2.3561944" />
+    <xacro:arg name="qb_tcp_rpy" default="0.785398 -1.5707963 2.3561944" />
     <xacro:include filename="$(find franka_description)/robots/common/utils.xacro" />
     <xacro:include filename="$(find franka_description)/robots/common/franka_arm.xacro" />
@@ -31,7 +31,27 @@
     </xacro:if>
     <xacro:if value="$(arg use_qbhand)">
+      <xacro:arg name="compensation_qb_tcp_xyz" default="-0.20 -0.003 0.053"/>
+      <xacro:arg name="qb_mass" default="0.3735"/>
+      <joint name="EE_fix_joint" type="fixed">
+	      <origin xyz="0 0 0" rpy="0 0 -0.785398"/>
+	      <parent link="panda_link8" />
+	      <child link="EE_fix_link" />
+      </joint>
+      <link name="EE_fix_link">
+        <inertial>
+          <origin xyz="0 0 0"/>
+          <mass value="0.0"/>
+          <inertia ixx="0.0" ixy="0" ixz="0" iyy="0.0" iyz="0" izz="0.0"/>
+        </inertial>
+        <visual>
+          <geometry>
+            <box size="0.05 0.05 0.05"/>
+          </geometry>
+          <material name="gray"/>
+        </visual>
+      </link>
       <joint name="mass_compensation_joint" type="fixed">
-	      <origin xyz="-0.12 0 0.05" rpy="0 0 0"/>
-	      <parent link="panda_link8" />
+	      <origin xyz="$(arg compensation_qb_tcp_xyz)" rpy="0 0 0"/>
+	      <parent link="EE_fix_link" />
 	      <child link="mass_compensation_link" />
       </joint>
@@ -39,19 +59,13 @@
         <inertial>
           <origin xyz="0 0 0"/>
-          <mass value="0.76"/>
+          <mass value="$(arg qb_mass)"/>
           <inertia ixx="0.01" ixy="0" ixz="0" iyy="0.01" iyz="0" izz="0.01"/>
         </inertial>
         <visual>
           <geometry>
-            <box size="0.1 0.1 0.1"/>
+            <box size="0.05 0.05 0.05"/>
           </geometry>
-          <material name="gray">
-    +	  </material>
+          <material name="gray"/>
         </visual>
-        <collision>
-          <geometry>
-            <box size="0.1 0.1 0.1"/>
-          </geometry>
-        </collision>
       </link>
       <xacro:include filename="$(find franka_qbhand)/urdf/softhands.xacro"/>
@@ -59,7 +73,7 @@
         type = "right"
         version = "v2.0_simple"
-        parent = "panda_link8"
+        parent = "EE_fix_link"
         position ="$(arg qb_tcp_xyz)"
-        orientation ="$(arg qb_tcp_xyz)"
+        orientation ="$(arg qb_tcp_rpy)"
         operation_mode = "0"
         translation="0.0036"
